File: hardware/KiCad/BigDripperController.kicad_sch (KiCad schematic)
At the start: 94 parts, among them Q1 IRL540NPBF, Q10 IRL540NPBF, Q11 IRL540NPBF, Q12 IRL540NPBF, Q13 IRL540NPBF, Q14 IRL540NPBF, Q15 IRL540NPBF, Q16 IRL540NPBF, Q17 TL2575-05IKV, Q2 IRL540NPBF, Q3 IRL540NPBF, Q4 IRL540NPBF, Q5 IRL540NPBF, Q6 IRL540NPBF, Q7 IRL540NPBF, Q8 IRL540NPBF, Q9 IRL540NPBF, U18 SN74HCT125NE4, U2 SN74HCT125NE4, U3 SN74HCT125NE4, U4 SN74HCT125NE4, U5 SN74HCT125NE4

Commit message: Added updated schematic and layout.
* Added production files for 1.1
Parts:
- added C6: 100uF, hackheim:CAP ALUM 10UF 20% 25V RADIAL TH - WÜRTH - 860020472003, symbol Device:C_Polarized
- added C7: 330uF, hackheim:CAP ALUM 10UF 20% 25V RADIAL TH - WÜRTH - 860020472003, symbol Device:C_Polarized
- added CR2, CR3, CR4: 1N5819, hackheim:DO-41_STM, symbol hackheim:1N5819
- added D20, D21, D22, D23, D24, D25, D26, D27, D28, D29, D30, D31, D32, D33, D34, D35, D36: LED, LED_THT:LED_D5.0mm, symbol Device:LED
- added L2: PE-52627NL, hackheim:PE52627NL, symbol hackheim:PE-52627NL
- added Q18: TL2575-05IKV, hackheim:TL2575-05IKV, symbol hackheim:TL2575-05IKV
- added R40, R41, R42, R43, R44, R45, R46, R47, R48, R49, R50, R51, R52, R53, R54, R55: 2k, Resistor_THT:R_Axial_DIN0207_L6.3mm_D2.5mm_P10.16mm_Horizontal, symbol Device:R
- added R56: R, Resistor_THT:R_Axial_DIN0207_L6.3mm_D2.5mm_P10.16mm_Horizontal, symbol Device:R
- CR1: footprint (none) -> hackheim:DO-41_STM
Connections:
- net 12V: now also CR2.2, CR3.2, R40.1, R41.1, R42.1, R43.1, R44.1, R45.1, R46.1, R47.1, R48.1, R49.1, R50.1, R51.1, R52.1, R53.1, R54.1, R55.1; no longer C1.1, Q17.1 (VIN)
- net COIL1: now also U1.15 (GPIO9); no longer U1.25 (GPIO19)
- net COIL10: now also U1.39 (GPIO42); no longer U1.34 (GPIO37)
- net COIL11: now also U1.38 (GPIO41); no longer U1.35 (GPIO38)
- net COIL12: now also U1.37 (GPIO40); no longer U1.36 (GPIO39)
- net COIL13: now also U1.36 (GPIO39); no longer U1.37 (GPIO40)
- net COIL14: now also U1.35 (GPIO38); no longer U1.38 (GPIO41)
- net COIL15: now also U1.12 (GPIO8); no longer U1.39 (GPIO42)
- net COIL16: now also U1.7 (GPIO7); no longer U1.40 (GPIO2)
- net COIL2: now also U1.17 (GPIO11); no longer U1.26 (GPIO20)
- net COIL3: now also U1.16 (GPIO10); no longer U1.27 (GPIO21)
- net COIL4: now also U1.18 (GPIO12); no longer U1.28 (GPIO47)
- net COIL5: now also U1.20 (GPIO14); no longer U1.29 (GPIO48)
- net COIL6: now also U1.19 (GPIO13); no longer U1.30 (GPIO45)
- net COIL7: now also U1.41 (GPIO1); no longer U1.31 (GPIO0)
- net COIL8: now also U1.6 (GPIO6); no longer U1.32 (GPIO35)
- net COIL9: now also U1.40 (GPIO2); no longer U1.33 (GPIO36)
- net GND: now also J4.5 (GND), J4.6 (GND), C6.2, C7.2, CR4.2, D36.1 (K), Q18.3 (GND), Q18.5 (~{ON}/OFF); no longer J4.16 (GND), J4.3 (GND)
- net C5: now reaches D5.2 (A), J2.10 (C5B), Q5.2 (D)
- net C5: now also D24.1 (K)
- net C11: now reaches D11.2 (A), J2.22 (C11B), Q11.2 (D)
- net C11: now also D30.1 (K)
- net C16: now reaches D16.2 (A), J2.32 (C16B), Q16.2 (D)
- net C16: now also D35.1 (K)
- net C4: now reaches D4.2 (A), J2.8 (C4B), Q4.2 (D)
- net C4: now also D23.1 (K)
- net C12: now reaches D12.2 (A), J2.24 (C12B), Q12.2 (D)
- net C12: now also D31.1 (K)
- net C9: now reaches D9.2 (A), J2.18 (C9B), Q9.2 (D)
- net C9: now also D28.1 (K)
- net C8: now reaches D8.2 (A), J2.16 (C8B), Q8.2 (D)
- net C8: now also D27.1 (K)
- net C1: now reaches D1.2 (A), J2.2 (C1B), Q1.2 (D)
- net C1: now also D20.1 (K)
- net C15: now reaches D15.2 (A), J2.30 (C15B), Q15.2 (D)
- net C15: now also D34.1 (K)
- net C10: now reaches D10.2 (A), J2.20 (C10B), Q10.2 (D)
- net C10: now also D29.1 (K)
- net C3: now reaches D3.2 (A), J2.6 (C3B), Q3.2 (D)
- net C3: now also D22.1 (K)
- net C2: now reaches D2.2 (A), J2.4 (C2B), Q2.2 (D)
- net C2: now also D21.1 (K)
- net C6: now reaches D6.2 (A), J2.12 (C6B), Q6.2 (D)
- net C6: now also D25.1 (K)
- net C14: now reaches D14.2 (A), J2.28 (C14A), Q14.2 (D)
- net C14: now also D33.1 (K)
- net C13: now reaches D13.2 (A), J2.26 (C13B), Q13.2 (D)
- net C13: now also D32.1 (K)
- net C7: now reaches D7.2 (A), J2.14 (C7B), Q7.2 (D)
- net C7: now also D26.1 (K)
- net GPIO1 renamed GPIO47
- net GPIO47: now also U1.28 (GPIO47); no longer U1.41 (GPIO1)
- removed net GPIO10: J4.9 (GPIO10), U1.16 (GPIO10)
- removed net GPIO11: J4.10 (GPIO11), U1.17 (GPIO11)
- removed net GPIO12: J4.11 (GPIO12), U1.18 (GPIO12)
- removed net GPIO13: J4.12 (GPIO13), U1.19 (GPIO13)
- removed net GPIO14: J4.13 (GPIO14), U1.20 (GPIO14)
- net GPIO43: no longer names the net of U1.43 (GPIO43)
- net GPIO43: no longer J4.14 (GPIO43)
- net GPIO44: no longer names the net of U1.42 (GPIO44)
- net GPIO44: no longer J4.15 (GPIO44)
- removed net GPIO6: J4.5 (GPIO6), U1.6 (GPIO6)
- removed net GPIO7: J4.6 (GPIO7), U1.7 (GPIO7)
- removed net GPIO8: J4.7 (GPIO8), U1.12 (GPIO8)
- removed net GPIO9: J4.8 (GPIO9), U1.15 (GPIO9)
- new net: D21.2 (A), R41.2
- new net: CR4.1, L2.1 (1+), Q18.2 (OUTPUT)
- new net: C1.1, CR2.1, Q17.1 (VIN)
- new net: D23.2 (A), R43.2
- new net: D24.2 (A), R44.2
- new net: D22.2 (A), R42.2
- new net: D27.2 (A), R47.2
- new net: D25.2 (A), R45.2
- new net: C6.1, CR3.1, Q18.1 (VIN)
- new net: D33.2 (A), R53.2
- new net: D34.2 (A), R54.2
- new net: D28.2 (A), R48.2
- new net: D30.2 (A), R50.2
- new net: D31.2 (A), R51.2
- new net: D32.2 (A), R52.2
- new net: D29.2 (A), R49.2
- new net: D20.2 (A), R40.2
- new net: D35.2 (A), R55.2
- new net: D26.2 (A), R46.2
- new net: D36.2 (A), R56.2
- new net GPIO21: J4.3 (GPIO21), U1.27 (GPIO21)
- new net NEOPIXEL_5V: C7.1, J5.10 (5V), J5.11 (5V), J5.12 (5V), J5.9 (5V), L2.2 (1-), Q18.4 (FEEDBACK), R56.1
Other:
- moved on the sheet: J3, R33, R34, R35, R36, U1, U18
